Commit message: prove IMU

File: src/ultron_description/urdf/ultron.urdf.xacro (robot description, xacro)
@@ -2,4 +2,13 @@
  <!-- Tutto in metri-->
 <robot name="ultron_robot" xmlns:xacro="http://ros.org/wiki/xacro">
+  <xacro:arg name="laser_enabled" default="false" />
+  <xacro:arg name="laser_xyz" default="$(optenv HUSKY_LMS1XX_XYZ 0.2206 0.0 0.00635)" />
+  <xacro:arg name="laser_rpy" default="$(optenv HUSKY_LMS1XX_RPY 0.0 0.0 0.0)" />
+  <xacro:arg name="kinect_enabled" default="false" />
+  <xacro:arg name="kinect_xyz" default="$(optenv HUSKY_KINECT_XYZ 0 0 0)" />
+  <xacro:arg name="kinect_rpy" default="$(optenv HUSKY_KINECT_RPY 0 0.18 3.14)" />
+  <xacro:arg name="imu_enabled" default="true" />
+  <xacro:arg name="robot_namespace" default="/" />
+  <xacro:arg name="urdf_extras" default="empty.urdf" />
   <!-- Included URDF/XACRO Files -->
 <!--  <xacro:include filename="$(find ultron_description)/urdf/decorations.urdf.xacro" />-->
@@ -26,5 +35,4 @@
   <xacro:property name="wheel_length" value="0.025" />
   <xacro:property name="wheel_radius" value="0.075" />
-  <xacro:macro name="ultron_robot">
     <!-- Base link is the center of the robot's bottom plate -->
     <link name="base_link">
@@ -110,7 +118,17 @@
     <!-- Can be modified with environment variables in /etc/ros/setup.bash -->
     <xacro:if value="$(arg imu_enabled)">
-        <link name="imu_link"/>
+        <link name="imu_link">
+	        <visual>
+	                <origin xyz="0 0 -0.015" rpy="0 0 0" />
+                        <geometry>
+                                <box size="0.03 0.03 0.03"/>
+                        </geometry>
+                         <material name="yellow">
+                  		<color rgba="1 1 0 1"/>
+		         </material>
+                </visual>
+        </link>
         <joint name="imu_joint" type="fixed">
-                <origin xyz="$(optenv ultron_IMU_XYZ 0.19 0 0.149)" rpy="$(optenv ultron_IMU_RPY 0 -1.5708 3.1416)" />
+                <origin xyz="0 0 -${base_z_size}" rpy="0 0 0" />
                 <parent link="base_link" />
                 <child link="imu_link" />
@@ -133,15 +151,4 @@
     </xacro:ultron_wheel>
    <!-- <xacro:ultron_decorate />-->
-    <xacro:if value="$(arg ur5_enabled)">
-      <xacro:property name="reflect" value="-1" />
-      <!-- Spawn arm -->
-      <xacro:ur5_robot prefix="ur5_arm_" joint_limited="true"/>
-      <!-- Join arm -->
-      <joint name="ur5_arm_base" type="fixed">
-        <parent link="top_plate_link" />
-        <child link="ur5_arm_base_link" />
-        <origin xyz="0.3058 0 0.0065" rpy="0.0 0.0 -1.57" />
-      </joint>
-    </xacro:if>
     <xacro:if value="$(arg laser_enabled)">
       <sick_lms1xx_mount prefix="base" topic="scan"/>
@@ -154,14 +161,47 @@
     </xacro:if>
     <xacro:if value="$(arg kinect_enabled)">
-      <xacro:sensor_arch prefix="" parent="top_plate_link">
-        <origin xyz="-0.35 0 0.51" rpy="0 0 -3.14"/>
-      </xacro:sensor_arch>
-      <joint name="kinect_frame_joint" type="fixed">
-        <origin xyz="$(optenv ultron_KINECT_XYZ 0 0 0)" rpy="$(optenv ultron_KINECT_RPY 0 0.18 3.14)" />
-        <parent link="sensor_arch_mount_link"/>
-        <child link="camera_link"/>
-      </joint>
-      <xacro:kinect_camera prefix="camera"/>
-    </xacro:if>
-  </xacro:macro>
+    <xacro:sensor_arch prefix="" parent="top_plate_link">
+      <origin xyz="-0.35 0 0.51" rpy="0 0 -3.14"/>
+    </xacro:sensor_arch>
+    <joint name="kinect_frame_joint" type="fixed">
+      <origin xyz="$(arg kinect_xyz)" rpy="$(arg kinect_rpy)" />
+      <parent link="sensor_arch_mount_link"/>
+      <child link="camera_link"/>
+    </joint>
+    <xacro:kinect_camera prefix="camera" robot_namespace="$(arg robot_namespace)"/>
+  </xacro:if>
+  <gazebo>
+    <plugin name="gazebo_ros_control" filename="libgazebo_ros_control.so">
+      <robotNamespace>$(arg robot_namespace)</robotNamespace>
+    </plugin>
+  </gazebo>
+  <gazebo>
+    <plugin name="imu_controller" filename="libhector_gazebo_ros_imu.so">
+      <robotNamespace>$(arg robot_namespace)</robotNamespace>
+      <updateRate>50.0</updateRate>
+      <bodyName>base_link</bodyName>
+      <topicName>imu/data</topicName>
+      <accelDrift>0.005 0.005 0.005</accelDrift>
+      <accelGaussianNoise>0.005 0.005 0.005</accelGaussianNoise>
+      <rateDrift>0.005 0.005 0.005 </rateDrift>
+      <rateGaussianNoise>0.005 0.005 0.005 </rateGaussianNoise>
+      <headingDrift>0.005</headingDrift>
+      <headingGaussianNoise>0.005</headingGaussianNoise>
+    </plugin>
+  </gazebo>
+  <gazebo>
+    <plugin name="gps_controller" filename="libhector_gazebo_ros_gps.so">
+      <robotNamespace>$(arg robot_namespace)</robotNamespace>
+      <updateRate>40</updateRate>
+      <bodyName>base_link</bodyName>
+      <frameId>base_link</frameId>
+      <topicName>navsat/fix</topicName>
+      <velocityTopicName>navsat/vel</velocityTopicName>
+      <referenceLatitude>49.9</referenceLatitude>
+      <referenceLongitude>8.9</referenceLongitude>
+      <referenceHeading>0</referenceHeading>
+      <referenceAltitude>0</referenceAltitude>
+      <drift>0.0001 0.0001 0.0001</drift>
+    </plugin>
+  </gazebo>
 </robot>

Commit message: cf

File: src/ultron_description/urdf/ultron.urdf.xacro (robot description, xacro)
@@ -115,6 +115,6 @@
       <child link="inertial_link" />
     </joint>
-    <!-- IMU Link is the standard mounting position for the UM6 IMU.-->
-    <!-- Can be modified with environment variables in /etc/ros/setup.bash -->
+    <!-- IMU Link is the standard mounting position for the  IMU.-->
+    <!-- Il sistena di asse e' diverso yaw = M_PI-->
     <xacro:if value="$(arg imu_enabled)">
         <link name="imu_link">
@@ -130,5 +130,5 @@
         </link>
         <joint name="imu_joint" type="fixed">
-                <origin xyz="0 0 -${base_z_size}" rpy="0 0 0" />
+                <origin xyz="0 0 -${base_z_size + 0.01}" rpy="0 0 -${M_PI}" />
                 <parent link="base_link" />
                 <child link="imu_link" />
