Commit message: model

File: src/ultron_description/urdf/description.xacro (robot description, xacro)
@@ -3,6 +3,6 @@
   <xacro:arg name="laser_enabled" default="false" />
   <xacro:arg name="ur5_enabled" default="false" />
-  <xacro:arg name="kinect_enabled" default="false" />
-  <xacro:arg name="imu_enabled" default="false" />
+  <xacro:arg name="kinect_enabled" default="true" />
+  <xacro:arg name="imu_enabled" default="true" />
   <xacro:include filename="$(find ultron_description)/urdf/ultron.urdf.xacro" />
   <xacro:ultron_robot />

File: src/ultron_description/urdf/ultron.urdf.xacro (robot description, xacro)
@@ -6,6 +6,7 @@
   <xacro:arg name="laser_rpy" default="$(optenv HUSKY_LMS1XX_RPY 0.0 0.0 0.0)" />
   <xacro:arg name="kinect_enabled" default="false" />
-  <xacro:arg name="kinect_xyz" default="0 0 0)" />
-  <xacro:arg name="kinect_rpy" default="0 0.18 3.14)" />
+  <xacro:arg name="kinect_xyz" default="0 0 0.03" />
+  <xacro:arg name="kinect_rpy" default="0 0 3.1415" />
+  <!--<xacro:arg name="kinect_rpy" default="0 0.18 3.1415" />-->
   <xacro:arg name="imu_enabled" default="true" />
   <xacro:arg name="robot_namespace" default="/" />
@@ -27,5 +28,5 @@
   <property name="border_y_size" value="0.06" />
   <!-- Top Plate -->
-  <property name="top_plate_xy_ray" value="0.13" />
+  <property name="top_plate_xy_ray" value="0.155" />
   <property name="top_plate_z_size" value="0.012" />
   <property name="top_plate_z_pos" value="0.253" />
@@ -188,10 +189,10 @@
     </xacro:if>
     <xacro:if value="$(arg kinect_enabled)">
-    <xacro:sensor_arch prefix="" parent="top_plate_link">
-      <origin xyz="-0.35 0 0.51" rpy="0 0 -3.14"/>
-    </xacro:sensor_arch>
+   <!-- <xacro:sensor_arch prefix="" parent="top_plate_link">
+      <origin xyz="0 0 0" rpy="0 0 -3.14"/>
+    </xacro:sensor_arch>-->
     <joint name="kinect_frame_joint" type="fixed">
       <origin xyz="$(arg kinect_xyz)" rpy="$(arg kinect_rpy)" />
-      <parent link="sensor_arch_mount_link"/>
+      <parent link="top_plate_link"/>
       <child link="camera_link"/>
     </joint>

Commit message: phantom

File: src/ultron_description/urdf/description.xacro (robot description, xacro)
@@ -3,6 +3,7 @@
   <xacro:arg name="laser_enabled" default="false" />
   <xacro:arg name="ur5_enabled" default="false" />
-  <xacro:arg name="kinect_enabled" default="true" />
-  <xacro:arg name="imu_enabled" default="true" />
+  <xacro:arg name="kinect_enabled" default="false" />
+  <xacro:arg name="imu_enabled" default="false" />
+  <xacro:arg name="zed_enabled" default="true" />
   <xacro:include filename="$(find ultron_description)/urdf/ultron.urdf.xacro" />
   <xacro:ultron_robot />

File: src/ultron_description/urdf/ultron.urdf.xacro (robot description, xacro)
@@ -6,4 +6,5 @@
   <xacro:arg name="laser_rpy" default="$(optenv HUSKY_LMS1XX_RPY 0.0 0.0 0.0)" />
   <xacro:arg name="kinect_enabled" default="false" />
+  <xacro:arg name="zed_enabled" default="true" />
   <!--<xacro:arg name="kinect_rpy" default="0 0.18 3.1415" />-->
   <xacro:arg name="imu_enabled" default="true" />
@@ -17,5 +18,10 @@
   <xacro:include filename="$(find ultron_description)/urdf/accessories/sensor_arch.urdf.xacro"/>
   <xacro:include filename="$(find ur_description)/urdf/ur5.urdf.xacro" />
-  <property name="M_PI" value="3.14159"/>
+  <xacro:include filename="$(find ultron_description)/urdf/zed.urdf.xacro" />
+  <xacro:include filename="$(find ultron_description)/urdf/imu.urdf.xacro" />
+  <!-- Global properties -->
+  <xacro:property name="path_meshes" value="package://ultron_description/meshes"/>
+  <xacro:property name="M_PI" value="3.14159"/>
+  <!-- Global properties -->
   <!-- Base Size -->
   <property name="base_x_size" value="0.45" />
@@ -26,7 +32,12 @@
   <property name="border_y_size" value="0.06" />
   <!-- Top Plate -->
-  <property name="top_plate_xy_ray" value="0.155" />
-  <property name="top_plate_z_size" value="0.012" />
-  <property name="top_plate_z_pos" value="0.253" />
+  <property name="top_plate_x_size" value="0.4" />
+  <property name="top_plate_y_size" value="0.34" />
+  <property name="top_plate_z_size" value="0.02" />
+  <property name="top_plate_z_pos" value="0.14" />
+  <!-- Verical bar Size -->
+  <property name="bar_x_size" value="0.02" />
+  <property name="bar_y_size" value="0.04" />
+  <property name="bar_z_size" value="1" />
   <!-- Wheel Mounting Positions -->
   <!-- dimensione del perimetro di attacco delle ruote-->
@@ -83,5 +94,5 @@
     <link name="base_link_platform_right">
         <visual>
-	        <origin xyz="0 0 -${base_z_size/2}" rpy="0 0 0" />
+                <origin xyz="0 0 -${base_z_size/2}" rpy="0 0 0" />
                 <geometry>
                         <box size="${border_x_size} ${border_y_size} ${base_z_size}"/>
@@ -104,7 +115,7 @@
     <link name="top_plate_link">
         <visual>
-	        <origin xyz="0 0 -${top_plate_z_size/2}" rpy="0 0 0" />
-                <geometry>
-                        <cylinder length="${top_plate_z_size}" radius="${top_plate_xy_ray}"/>
+                <origin xyz="0 0 -${top_plate_z_size/2}" rpy="0 0 0" />
+                <geometry>
+                        <box size="${top_plate_x_size} ${top_plate_y_size} ${top_plate_z_size}"/>
                 </geometry>
                  <material name="gray">
@@ -115,5 +126,5 @@
                 <origin xyz="0 0 -${top_plate_z_size/2}" rpy="0 0 0" />
                 <geometry>
-                         <cylinder length="${top_plate_z_size}" radius="${top_plate_xy_ray}"/>
+                         <box size="${top_plate_x_size} ${top_plate_y_size} ${top_plate_z_size}"/>
                 </geometry>
       </collision>
@@ -131,4 +142,29 @@
       <child link="base_footprint" />
     </joint>
+<!-- barra verticale -->
+<link name="bar_link">
+    <visual>
+        <origin xyz="0 0 ${bar_z_size/2}" rpy="0 0 0" />
+        <geometry>
+              <box size="${bar_x_size} ${bar_y_size} ${bar_z_size}"/>
+        </geometry>
+        <material name="black">
+          <color rgba="0 1 0 1"/>
+        </material>
+      </visual>
+  </link>
+  <joint name="bar_join" type="fixed">
+    <!--<xacro:insert_block name="joint_pose"/>-->
+    <parent link="base_link" />
+    <child link="bar_link" />
+    <origin xyz="${-base_x_size/2 + bar_x_size} 0 0" rpy="0 0 0" />
+    <axis xyz="0 0 0" />
+  </joint>
+<!-- barra verticale -->
+  <!-- ZED -->
+  <xacro:zed_lidar parent="bar_link">
+    <origin xyz="${-bar_x_size/2} 0 0.675" rpy="0 0 0" />
+  </xacro:zed_lidar>
+  <!-- ZED - END -->
     <!-- Interial link stores the robot's inertial information -->
     <link name="inertial_link">
@@ -147,13 +183,13 @@
     <!-- Il sistena di asse e' diverso yaw = M_PI-->
     <xacro:if value="$(arg imu_enabled)">
-        <link name="imu_link">
-	        <visual>
-	                <origin xyz="0 0 -0.015" rpy="0 0 0" />
+       <!--<link name="imu_link">
+                <visual>
+                        <origin xyz="0 0 -0.015" rpy="0 0 0" />
                         <geometry>
                                 <box size="0.03 0.03 0.03"/>
                         </geometry>
                          <material name="yellow">
-                  		<color rgba="1 1 0 1"/>
-		         </material>
+                                <color rgba="1 1 0 1"/>
+                         </material>
                 </visual>
         </link>
@@ -162,5 +198,11 @@
                 <parent link="base_link" />
                 <child link="imu_link" />
-       </joint>
+       </joint>-->
+       <!-- IMU -->
+        <xacro:imu parent="base_link">
+         <!-- <origin xyz="0 0 0" rpy="0 ${M_PI/2} 0" /> -->
+          <origin xyz="0 0 0" rpy="0  0 0" />
+        </xacro:imu>
+        <!-- IMU -->
        <gazebo reference="imu_link">
        </gazebo>
