Commit message: slam

File: src/ultron_description/urdf/accessories/kinect_camera.urdf.xacro (robot description, xacro)
@@ -1,5 +1,30 @@
 <?xml version="1.0"?>
+<!--
+Copyright (c) 2013, Goncalo Cabrita, ISR University of Coimbra
+Copyright (c) 2016, Clearpath Robotics
+All rights reserved.
+Redistribution and use in source and binary forms, with or without
+modification, are permitted provided that the following conditions are met:
+    * Redistributions of source code must retain the above copyright
+      notice, this list of conditions and the following disclaimer.
+    * Redistributions in binary form must reproduce the above copyright
+      notice, this list of conditions and the following disclaimer in the
+      documentation and/or other materials provided with the distribution.
+    * Neither the name of Clearpath Robotics nor the
+      names of its contributors may be used to endorse or promote products
+      derived from this software without specific prior written permission.
+THIS SOFTWARE IS PROVIDED BY THE COPYRIGHT HOLDERS AND CONTRIBUTORS "AS IS" AND
+ANY EXPRESS OR IMPLIED WARRANTIES, INCLUDING, BUT NOT LIMITED TO, THE IMPLIED
+WARRANTIES OF MERCHANTABILITY AND FITNESS FOR A PARTICULAR PURPOSE ARE
+DISCLAIMED. IN NO EVENT SHALL THE COPYRIGHT HOLDERS BE LIABLE FOR ANY
+DIRECT, INDIRECT, INCIDENTAL, SPECIAL, EXEMPLARY, OR CONSEQUENTIAL DAMAGES
+(INCLUDING, BUT NOT LIMITED TO, PROCUREMENT OF SUBSTITUTE GOODS OR SERVICES;
+LOSS OF USE, DATA, OR PROFITS; OR BUSINESS INTERRUPTION) HOWEVER CAUSED AND
+ON ANY THEORY OF LIABILITY, WHETHER IN CONTRACT, STRICT LIABILITY, OR TORT
+(INCLUDING NEGLIGENCE OR OTHERWISE) ARISING IN ANY WAY OUT OF THE USE OF THIS
+SOFTWARE, EVEN IF ADVISED OF THE POSSIBILITY OF SUCH DAMAGE.
+-->
 <robot xmlns:xacro="http://ros.org/wiki/xacro" name="kinect_camera">
-  <xacro:macro name="kinect_camera" params="prefix:=camera">
+  <xacro:macro name="kinect_camera" params="prefix:=camera robot_namespace:=/">
     <!-- Create kinect reference frame -->
     <!-- Add mesh for kinect -->
@@ -18,4 +43,47 @@
       </collision>
     </link>
+    <joint name="${prefix}_optical_joint" type="fixed">
+      <origin xyz="0 0 0" rpy="-1.5708 0 -1.5708"/>
+      <parent link="${prefix}_link"/>
+      <child link="${prefix}_frame_optical"/>
+    </joint>
+    <link name="${prefix}_frame_optical"/>
+    <gazebo reference="${prefix}_link">
+      <sensor type="depth" name="${prefix}">
+        <always_on>true</always_on>
+        <update_rate>20.0</update_rate>
+        <camera>
+          <horizontal_fov>${60.0*M_PI/180.0}</horizontal_fov>
+          <image>
+            <format>R8G8B8</format>
+            <width>640</width>
+            <height>480</height>
+          </image>
+          <clip>
+            <near>0.05</near>
+            <far>8.0</far>
+          </clip>
+        </camera>
+        <plugin name="kinect_${prefix}_controller" filename="libgazebo_ros_openni_kinect.so">
+          <cameraName>${prefix}</cameraName>
+          <alwaysOn>true</alwaysOn>
+          <updateRate>10</updateRate>
+          <imageTopicName>rgb/image_raw</imageTopicName>
+          <depthImageTopicName>depth/image_raw</depthImageTopicName>
+          <pointCloudTopicName>depth/points</pointCloudTopicName>
+          <cameraInfoTopicName>rgb/camera_info</cameraInfoTopicName>
+          <depthImageCameraInfoTopicName>depth/camera_info</depthImageCameraInfoTopicName>
+          <frameName>${prefix}_frame_optical</frameName>
+          <baseline>0.1</baseline>
+          <distortion_k1>0.0</distortion_k1>
+          <distortion_k2>0.0</distortion_k2>
+          <distortion_k3>0.0</distortion_k3>
+          <distortion_t1>0.0</distortion_t1>
+          <distortion_t2>0.0</distortion_t2>
+          <pointCloudCutoff>0.4</pointCloudCutoff>
+          <robotNamespace>${robot_namespace}</robotNamespace>
+        </plugin>
+      </sensor>
+    </gazebo>
   </xacro:macro>
 </robot>

File: src/ultron_description/urdf/accessories/sensor_arch.urdf.xacro (robot description, xacro)
@@ -7,5 +7,5 @@
              <visual>
                  <geometry>
-                     <mesh filename="package://ultron_description/meshes/accessories/${size}_mm_sensor_arch.dae" />
+                     <mesh filename="package://husky_description/meshes/accessories/${size}_mm_sensor_arch.dae" />
                  </geometry>
              </visual>
@@ -13,5 +13,5 @@
                  <origin xyz="0 0 0" rpy="0 0 0"/>
                  <geometry>
-                     <mesh filename="package://ultron_description/meshes/accessories/${size}_mm_sensor_arch.dae" />
+                     <mesh filename="package://husky_description/meshes/accessories/${size}_mm_sensor_arch.dae" />
                  </geometry>
              </collision>

File: src/ultron_description/urdf/accessories/sick_lms1xx_mount.urdf.xacro (robot description, xacro)
@@ -1,7 +1,31 @@
 <?xml version="1.0"?>
+<!--
+Copyright (c) 2013, Goncalo Cabrita, ISR University of Coimbra
+Copyright (c) 2014, 2015 Clearpath Robotics
+All rights reserved.
+Redistribution and use in source and binary forms, with or without
+modification, are permitted provided that the following conditions are met:
+    * Redistributions of source code must retain the above copyright
+      notice, this list of conditions and the following disclaimer.
+    * Redistributions in binary form must reproduce the above copyright
+      notice, this list of conditions and the following disclaimer in the
+      documentation and/or other materials provided with the distribution.
+    * Neither the name of Clearpath Robotics nor the
+      names of its contributors may be used to endorse or promote products
+      derived from this software without specific prior written permission.
+THIS SOFTWARE IS PROVIDED BY THE COPYRIGHT HOLDERS AND CONTRIBUTORS "AS IS" AND
+ANY EXPRESS OR IMPLIED WARRANTIES, INCLUDING, BUT NOT LIMITED TO, THE IMPLIED
+WARRANTIES OF MERCHANTABILITY AND FITNESS FOR A PARTICULAR PURPOSE ARE
+DISCLAIMED. IN NO EVENT SHALL THE COPYRIGHT HOLDERS BE LIABLE FOR ANY
+DIRECT, INDIRECT, INCIDENTAL, SPECIAL, EXEMPLARY, OR CONSEQUENTIAL DAMAGES
+(INCLUDING, BUT NOT LIMITED TO, PROCUREMENT OF SUBSTITUTE GOODS OR SERVICES;
+LOSS OF USE, DATA, OR PROFITS; OR BUSINESS INTERRUPTION) HOWEVER CAUSED AND
+ON ANY THEORY OF LIABILITY, WHETHER IN CONTRACT, STRICT LIABILITY, OR TORT
+(INCLUDING NEGLIGENCE OR OTHERWISE) ARISING IN ANY WAY OUT OF THE USE OF THIS
+SOFTWARE, EVEN IF ADVISED OF THE POSSIBILITY OF SUCH DAMAGE.
+-->
 <robot xmlns:xacro="http://ros.org/wiki/xacro">
   <xacro:include filename="$(find lms1xx)/urdf/sick_lms1xx.urdf.xacro" />
-  <xacro:macro name="sick_lms1xx_mount" params="prefix topic">
-  <sick_lms1xx frame="${prefix}_laser" topic="${topic}" />
+  <xacro:macro name="sick_lms1xx_mount" params="prefix">
     <link name="${prefix}_laser_mount">
       <visual>
@@ -9,5 +33,5 @@
         <geometry>
           <!-- Origin of this mesh is the base of the bracket. -->
-          <mesh filename="package://ultron_description/meshes/accessories/lms1xx_mount.dae" />
+          <mesh filename="package://husky_description/meshes/accessories/lms1xx_mount.dae" />
         </geometry>
       </visual>

File: src/ultron_description/urdf/ultron.urdf.xacro (robot description, xacro)
@@ -6,6 +6,6 @@
   <xacro:arg name="laser_rpy" default="$(optenv HUSKY_LMS1XX_RPY 0.0 0.0 0.0)" />
   <xacro:arg name="kinect_enabled" default="false" />
-  <xacro:arg name="kinect_xyz" default="$(optenv HUSKY_KINECT_XYZ 0 0 0)" />
-  <xacro:arg name="kinect_rpy" default="$(optenv HUSKY_KINECT_RPY 0 0.18 3.14)" />
+  <xacro:arg name="kinect_xyz" default="0 0 0)" />
+  <xacro:arg name="kinect_rpy" default="0 0.18 3.14)" />
   <xacro:arg name="imu_enabled" default="true" />
   <xacro:arg name="robot_namespace" default="/" />
@@ -26,4 +26,8 @@
   <property name="border_x_size" value="0.13" />
   <property name="border_y_size" value="0.06" />
+  <!-- Top Plate -->
+  <property name="top_plate_xy_ray" value="0.13" />
+  <property name="top_plate_z_size" value="0.012" />
+  <property name="top_plate_z_pos" value="0.253" />
   <!-- Wheel Mounting Positions -->
   <!-- dimensione del perimetro di attacco delle ruote-->
@@ -94,4 +98,27 @@
       <parent link="base_link" />
       <child link="base_link_platform_right" />
+    </joint>
+   <!-- pezzo su -->
+    <link name="top_plate_link">
+        <visual>
+	        <origin xyz="0 0 -${top_plate_z_size/2}" rpy="0 0 0" />
+                <geometry>
+                        <cylinder length="${top_plate_z_size}" radius="${top_plate_xy_ray}"/>
+                </geometry>
+                 <material name="gray">
+		  <color rgba="0.5 0.5 0.5 1"/>
+		</material>
+        </visual>
+        <collision>
+                <origin xyz="0 0 -${top_plate_z_size/2}" rpy="0 0 0" />
+                <geometry>
+                         <cylinder length="${top_plate_z_size}" radius="${top_plate_xy_ray}"/>
+                </geometry>
+      </collision>
+    </link>
+    <joint name="base_link_top_plate_link_joint" type="fixed">
+      <origin xyz="0 0 ${top_plate_z_pos}" rpy="0 0 0" />
+      <parent link="base_link" />
+      <child link="top_plate_link" />
     </joint>
     <!-- Base footprint is on the ground under the robot -->

Commit message: slam

File: src/ultron_description/urdf/accessories/kinect_camera.urdf.xacro (robot description, xacro)
@@ -32,5 +32,5 @@
       <origin xyz="0 0 0" rpy="0 0 0"/>
       <visual>
-        <origin xyz="0 0 0" rpy="0 0 ${M_PI/2}"/>
+        <origin xyz="0 0 0" rpy="0 0 0"/>
         <geometry>
           <mesh filename="package://ultron_description/meshes/accessories/kinect.dae" />

File: src/ultron_description/urdf/ultron.urdf.xacro (robot description, xacro)
@@ -6,6 +6,4 @@
   <xacro:arg name="laser_rpy" default="$(optenv HUSKY_LMS1XX_RPY 0.0 0.0 0.0)" />
   <xacro:arg name="kinect_enabled" default="false" />
-  <xacro:arg name="kinect_xyz" default="0 0 0.03" />
-  <xacro:arg name="kinect_rpy" default="0 0 3.1415" />
   <!--<xacro:arg name="kinect_rpy" default="0 0.18 3.1415" />-->
   <xacro:arg name="imu_enabled" default="true" />
@@ -40,4 +38,7 @@
   <xacro:property name="wheel_length" value="0.025" />
   <xacro:property name="wheel_radius" value="0.075" />
+  <!-- KInect Properties -->
+  <xacro:arg name="kinect_xyz" default="0 0 0.03" />
+  <xacro:arg name="kinect_rpy" default="0 0 0" />
     <!-- Base link is the center of the robot's bottom plate -->
     <link name="base_link">
